File: bms/bms.sch (KiCad schematic (older format))
At the start: 44 parts, among them Q1 2N3904

Commit message: bms updates
Parts:
- removed C? (x2): CP, symbol Device:CP
- added C? (x3): CP1_Small, symbol Device:CP1_Small
- added R? (x6): R, symbol Device:R
- added SW? (x4): SW_SPDT, symbol Switch:SW_SPDT
- added TH? (x3): Thermistor_NTC_US, symbol Device:Thermistor_NTC_US
- added U?: TPS2592xx, Package_SON:VSON-10-1EP_3x3mm_P0.5mm_EP1.65x2.4mm_ThermalVias, symbol Power_Management:TPS2592xx
Connections:
- wire segments 88 -> 125
Other:
- note added: "Overcurrent protection"
- moved on the sheet: BT?, R?, U?
