File: solenoidTrigger/solenoidTrigger.kicad_pcb (KiCad board)
At the start: 2 copper layers, 88.9 x 88.9 mm, 45 parts, among them J8 CONN_02X03, P1 OSTTC03, P2 OSTTC02, P3 OSTTC08, P4 OSTTC03, P5 OSTTC03, Q1 NMOS_CDS16, Q2 NMOS_CDS16, Q3 NMOS_CDS16, Q4 NMOS_CDS16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

Commit message: moved around oscillator
Parts:
- moved Y2 8.53 mm to (172.8, 81.5)
- moved C8 7.95 mm to (172.8, 78.2), turned to 0 degrees
- moved C6 6.89 mm to (172.9, 84.8)
Routing:
- net Net-(C6-Pad1): track 4.43 -> 0.00 mm
- net Net-(C8-Pad1): track 4.08 -> 0.37 mm
Changed lines of the file:
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@@
     (thickness 1.6)
     (drawings 8)
-    (tracks 114)
+    (tracks 109)
     (zones 0)
     (modules 45)
@@
   )
   (setup
-    (last_trace_width 0.254)
+    (last_trace_width 0.25)
     (user_trace_width 0.254)
     (user_trace_width 0.381)
@@
   )
   (module footprints:C_0805_OEM (layer F.Cu)
-    (at 171.45 78.105)
+    (at 172.9105 84.836)
     (descr "Capacitor SMD 0805, reflow soldering, AVX (see smccp.pdf)")
     (tags "capacitor 0805")
     (attr smd)
-    (fp_text reference C6 (at 0 -1.5) (layer F.SilkS)
+    (fp_text reference C6 (at 0 1.651) (layer F.SilkS)
       (effects (font (size 1 1) (thickness 0.15)))
     )
@@
   )
   (module footprints:C_0805_OEM (layer F.Cu)
-    (at 176.53 71.12 90)
+    (at 172.847 78.1685)
     (descr "Capacitor SMD 0805, reflow soldering, AVX (see smccp.pdf)")
     (tags "capacitor 0805")
     (attr smd)
-    (fp_text reference C8 (at 0 -1.5 90) (layer F.SilkS)
-      (effects (font (size 1 1) (thickness 0.15)))
-    )
-    (fp_text value C_30pF (at 0 1.75 90) (layer F.Fab) hide
+    (fp_text reference C8 (at 0 -1.5) (layer F.SilkS)
+      (effects (font (size 1 1) (thickness 0.15)))
+    )
+    (fp_text value C_30pF (at 0 1.75) (layer F.Fab) hide
       (effects (font (size 1 1) (thickness 0.15)))
     )
@@
     (fp_line (start 1 0.62) (end -1 0.62) (layer F.Fab) (width 0.1))
     (fp_line (start -1 0.62) (end -1 -0.62) (layer F.Fab) (width 0.1))
-    (pad 2 smd rect (at 1 0 90) (size 1 1.25) (layers F.Cu F.Paste F.Mask)
-      (net 1 GND))
-    (pad 1 smd rect (at -1 0 90) (size 1 1.25) (layers F.Cu F.Paste F.Mask)
+    (pad 2 smd rect (at 1 0) (size 1 1.25) (layers F.Cu F.Paste F.Mask)
+      (net 1 GND))
+    (pad 1 smd rect (at -1 0) (size 1 1.25) (layers F.Cu F.Paste F.Mask)
       (net 5 "Net-(C8-Pad1)"))
     (model /home/josh/Formula/OEM_Preferred_Parts/3DModels/C_0805_OEM/C_0805.wrl
@@
   )
   (module footprints:Crystal_SMD_FA238 (layer F.Cu)
-    (at 171.62 73.025 180)
+    (at 172.8265 81.4705 180)
     (descr "crystal Epson Toyocom FA-238 series http://www.mouser.com/ds/2/137/1721499-465440.pdf, hand-soldering, 3.2x2.5mm^2 package")
     (tags "SMD SMT crystal hand-soldering")
     (attr smd)
-    (fp_text reference Y2 (at -0.67564 -2.66192) (layer F.SilkS)
+    (fp_text reference Y2 (at -2.878 0.4445 270) (layer F.SilkS)
       (effects (font (size 1 1) (thickness 0.15)))
     )
@@
   (gr_line (start 191.77 132.08) (end 191.77 55.88) (layer Edge.Cuts) (width 0.2))
   (segment (start 110.779999 57.3913) (end 110.060099 57.3913) (width 0.254) (layer F.Cu) (net 0))
+  (via (at 176.022 78.1685) (size 0.8) (drill 0.4) (layers F.Cu B.Cu) (net 1))
+  (segment (start 173.847 78.1685) (end 176.022 78.1685) (width 0.254) (layer F.Cu) (net 1))
+  (via (at 176.0855 82.2325) (size 0.8) (drill 0.4) (layers F.Cu B.Cu) (net 1))
+  (segment (start 173.9105 82.2325) (end 176.0855 82.2325) (width 0.254) (layer F.Cu) (net 1))
   (segment (start 140.9065 73.4855) (end 140.9065 71.9455) (width 0.381) (layer F.Cu) (net 1))
   (segment (start 140.9065 71.9455) (end 140.9065 71.9455) (width 0.381) (layer F.Cu) (net 1))
@@
   (via (at 121.412 105.0925) (size 0.8) (drill 0.4) (layers F.Cu B.Cu) (net 1))
   (segment (start 119.872 105.0925) (end 121.412 105.0925) (width 0.381) (layer F.Cu) (net 1))
-  (segment (start 172.62 73.825) (end 172.45 73.995) (width 0.254) (layer F.Cu) (net 1))
-  (segment (start 172.72 73.825) (end 172.62 73.825) (width 0.254) (layer F.Cu) (net 1))
+  (segment (start 173.8265 82.2705) (end 173.6565 82.4405) (width 0.254) (layer F.Cu) (net 1))
+  (segment (start 173.9265 82.2705) (end 173.8265 82.2705) (width 0.254) (layer F.Cu) (net 1))
   (segment (start 170.749 110.4265) (end 172.339 110.4265) (width 0.254) (layer F.Cu) (net 1))
   (via (at 172.339 110.4265) (size 0.8) (drill 0.4) (layers F.Cu B.Cu) (net 1))
@@
   (via (at 168.275 105.537) (size 0.8) (drill 0.4) (layers F.Cu B.Cu) (net 1))
   (segment (start 168.275 103.462) (end 168.275 105.537) (width 0.254) (layer F.Cu) (net 1))
-  (segment (start 176.53 70.12) (end 174.26 70.12) (width 0.254) (layer F.Cu) (net 1))
-  (segment (start 174.26 70.12) (end 174.26 70.12) (width 0.254) (layer F.Cu) (net 1))
-  (via (at 174.26 70.12) (size 0.8) (drill 0.4) (layers F.Cu B.Cu) (net 1))
-  (via (at 168.275 72.39) (size 0.8) (drill 0.4) (layers F.Cu B.Cu) (net 1))
+  (via (at 169.4815 80.8355) (size 0.8) (drill 0.4) (layers F.Cu B.Cu) (net 1))
   (via (at 184.4675 83.693) (size 0.8) (drill 0.4) (layers F.Cu B.Cu) (net 1))
-  (via (at 174.625 78.105) (size 0.8) (drill 0.4) (layers F.Cu B.Cu) (net 1))
-  (via (at 173.99 75.565) (size 0.8) (drill 0.4) (layers F.Cu B.Cu) (net 1))
+  (via (at 176.0855 84.836) (size 0.8) (drill 0.4) (layers F.Cu B.Cu) (net 1))
   (segment (start 182.2925 83.693) (end 184.4675 83.693) (width 0.254) (layer F.Cu) (net 1))
-  (segment (start 170.355 72.39) (end 170.52 72.225) (width 0.254) (layer F.Cu) (net 1))
-  (segment (start 168.275 72.39) (end 170.355 72.39) (width 0.254) (layer F.Cu) (net 1))
-  (segment (start 172.72 74.295) (end 173.99 75.565) (width 0.254) (layer F.Cu) (net 1))
-  (segment (start 172.72 73.825) (end 172.72 74.295) (width 0.254) (layer F.Cu) (net 1))
-  (segment (start 172.45 78.105) (end 174.625 78.105) (width 0.254) (layer F.Cu) (net 1))
+  (segment (start 171.5615 80.8355) (end 171.7265 80.6705) (width 0.254) (layer F.Cu) (net 1))
+  (segment (start 169.4815 80.8355) (end 171.5615 80.8355) (width 0.254) (layer F.Cu) (net 1))
+  (segment (start 173.9265 82.2705) (end 173.9265 82.7405) (width 0.254) (layer F.Cu) (net 1))
+  (segment (start 173.9105 84.836) (end 176.0855 84.836) (width 0.254) (layer F.Cu) (net 1))
   (segment (start 167.445 83.42) (end 169.31 83.42) (width 0.254) (layer F.Cu) (net 1))
   (segment (start 169.31 83.42) (end 169.31 83.42) (width 0.254) (layer F.Cu) (net 1))
@@
   (segment (start 179.9725 78.806) (end 180.2925 78.486) (width 0.254) (layer F.Cu) (net 2))
   (segment (start 140.8905 84.328) (end 140.8905 84.453) (width 0.254) (layer F.Cu) (net 2))
-  (segment (start 170.52 78.035) (end 170.45 78.105) (width 0.254) (layer F.Cu) (net 4))
-  (segment (start 170.45 78.23) (end 170.45 78.105) (width 0.254) (layer F.Cu) (net 4))
-  (segment (start 170.52 73.825) (end 170.52 78.035) (width 0.254) (layer F.Cu) (net 4))
-  (segment (start 176.53 72.12) (end 176.405 72.12) (width 0.254) (layer F.Cu) (net 5))
-  (segment (start 172.72 72.225) (end 176.425 72.225) (width 0.254) (layer F.Cu) (net 5))
-  (segment (start 176.425 72.225) (end 176.53 72.12) (width 0.254) (layer F.Cu) (net 5))
-  (segment (start 172.62 72.225) (end 172.72 72.225) (width 0.254) (layer F.Cu) (net 5))
+  (segment (start 171.847 78.359) (end 171.847 78.234) (width 0.254) (layer F.Cu) (net 5))
+  (segment (start 171.742 78.254) (end 171.847 78.359) (width 0.254) (layer F.Cu) (net 5))
+  (segment (start 173.8265 80.6705) (end 173.9265 80.6705) (width 0.254) (layer F.Cu) (net 5))
   (segment (start 164.465 97.435) (end 164.465 101.262) (width 0.25) (layer F.Cu) (net 9))
   (segment (start 164.465 96.835) (end 164.465 97.435) (width 0.25) (layer F.Cu) (net 9))
